File: Panel/Panel.sch (KiCad schematic (older format))
At the start: 28 parts

Commit message: Panel
Bigger holes for pots
Parts:
- H22, H23, H24, H25, H26, H27, H28: footprint MountingHole:MountingHole_6.5mm -> MountingHole:MountingHole_8.4mm_M8
Changed lines of the file:
@@
 EESchema Schematic File Version 4
-LIBS:Panel-cache
 EELAYER 30 0
 EELAYER END
@@
 F 0 "H22" H 2350 7846 50  0000 L CNN
 F 1 "MountingHole" H 2350 7755 50  0000 L CNN
-F 2 "MountingHole:MountingHole_6.5mm" H 2250 7800 50  0001 C CNN
+F 2 "MountingHole:MountingHole_8.4mm_M8" H 2250 7800 50  0001 C CNN
 F 3 "~" H 2250 7800 50  0001 C CNN
 	1    2250 7800
@@
 F 0 "H23" H 2400 8446 50  0000 L CNN
 F 1 "MountingHole" H 2400 8355 50  0000 L CNN
-F 2 "MountingHole:MountingHole_6.5mm" H 2300 8400 50  0001 C CNN
+F 2 "MountingHole:MountingHole_8.4mm_M8" H 2300 8400 50  0001 C CNN
 F 3 "~" H 2300 8400 50  0001 C CNN
 	1    2300 8400
@@
 F 0 "H24" H 2450 9096 50  0000 L CNN
 F 1 "MountingHole" H 2450 9005 50  0000 L CNN
-F 2 "MountingHole:MountingHole_6.5mm" H 2350 9050 50  0001 C CNN
+F 2 "MountingHole:MountingHole_8.4mm_M8" H 2350 9050 50  0001 C CNN
 F 3 "~" H 2350 9050 50  0001 C CNN
 	1    2350 9050
@@
 F 0 "H25" H 2500 9596 50  0000 L CNN
 F 1 "MountingHole" H 2500 9505 50  0000 L CNN
-F 2 "MountingHole:MountingHole_6.5mm" H 2400 9550 50  0001 C CNN
+F 2 "MountingHole:MountingHole_8.4mm_M8" H 2400 9550 50  0001 C CNN
 F 3 "~" H 2400 9550 50  0001 C CNN
 	1    2400 9550
@@
 F 0 "H26" H 3650 7996 50  0000 L CNN
 F 1 "MountingHole" H 3650 7905 50  0000 L CNN
-F 2 "MountingHole:MountingHole_6.5mm" H 3550 7950 50  0001 C CNN
+F 2 "MountingHole:MountingHole_8.4mm_M8" H 3550 7950 50  0001 C CNN
 F 3 "~" H 3550 7950 50  0001 C CNN
 	1    3550 7950
@@
 F 0 "H27" H 3700 8496 50  0000 L CNN
 F 1 "MountingHole" H 3700 8405 50  0000 L CNN
-F 2 "MountingHole:MountingHole_6.5mm" H 3600 8450 50  0001 C CNN
+F 2 "MountingHole:MountingHole_8.4mm_M8" H 3600 8450 50  0001 C CNN
 F 3 "~" H 3600 8450 50  0001 C CNN
 	1    3600 8450
@@
 F 0 "H28" H 3850 9246 50  0000 L CNN
 F 1 "MountingHole" H 3850 9155 50  0000 L CNN
-F 2 "MountingHole:MountingHole_6.5mm" H 3750 9200 50  0001 C CNN
+F 2 "MountingHole:MountingHole_8.4mm_M8" H 3750 9200 50  0001 C CNN
 F 3 "~" H 3750 9200 50  0001 C CNN
 	1    3750 9200
