File: Panel/Panel Clean.kicad_pcb (KiCad board)
At the start: 2 copper layers, 70.8 x 128.5 mm, 28 parts

Commit message: Rename
Other:
- board text added: "NanoGris"
- board text removed: "NanoGrids"
Changed lines of the file:
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@@
     (effects (font (size 2 2) (thickness 0.5) italic))
   )
-  (gr_text NanoGrids (at 241.3 52.07 -90) (layer F.SilkS)
-    (effects (font (size 5 5) (thickness 0.75)))
+  (gr_text NanoGris (at 241.8334 53.4924 -90) (layer F.SilkS)
+    (effects (font (size 6 6) (thickness 1.5)))
   )
   (gr_text Tap (at 228.6 60.96) (layer F.SilkS)
