File: GridsNanoV3.sch (KiCad schematic (older format))
At the start: 112 parts, among them J10 Conn_01x12, J11 Conn_01x12, J12 Conn_02x05_Odd_Even, J13 Conn_01x10, J14 Conn_01x10, J15 Conn_01x10, J16 Conn_01x03, J7 Conn_01x10, Q1 2N3904, Q2 2N3904, U1 MCP6002_1, U2 MCP6002_1, U3 MCP6002_1, U4 L7805, U5 LM4040LP-5, U6 74HC595, X1 CV_X, Y1 CV_Y

Commit message: Updates 0.04
Updates for 0.04
Change footprint for pots
Added + sign for leds
Added usb side
Added Ground plane
Parts:
- D1: symbol GridsNanoV3-rescue:LED-Device -> Device:LED
- P_CH1, P_CH2, P_CH3, P_TEMPO1, P_X1, P_Y1: footprint Potentiometer_THT:Potentiometer_Alpha_RD901F-40-00D_Single_Vertical -> Potentiometer_THT:Potentiometer_Alps_RK09K_Single_Vertical
- P_RND1: footprint Potentiometer_THT:Potentiometer_Alpha_RD901F-40-00D_Single_Vertical -> Potentiometer_THT:Potentiometer_Alps_RK09L_Single_Vertical
Connections:
- net +5V: now also P_CH1.1, P_CH2.1, P_CH3.1, P_RND1.1, P_TEMPO1.1, P_X1.1, P_Y1.1; no longer P_CH1.3, P_CH2.3, P_CH3.3, P_RND1.3, P_TEMPO1.3, P_X1.3, P_Y1.3
- net GND: now also P_CH1.3, P_CH2.3, P_CH3.3, P_RND1.3, P_TEMPO1.3, P_X1.3, P_Y1.3; no longer P_CH1.1, P_CH2.1, P_CH3.1, P_RND1.1, P_TEMPO1.1, P_X1.1, P_Y1.1

Commit message: 0.04 Commit
Gerbers
Parts:
- P_CH1, P_CH2, P_CH3, P_TEMPO1, P_X1, P_Y1: footprint Potentiometer_THT:Potentiometer_Alps_RK09K_Single_Vertical -> Potentiometer_THT:Potentiometer_Alps_RK09L_Single_Vertical
Changed lines of the file:
@@
 F 0 "P_TEMPO1" H 8680 13896 50  0000 R CNN
 F 1 "10k" H 8680 13805 50  0000 R CNN
-F 2 "Potentiometer_THT:Potentiometer_Alps_RK09K_Single_Vertical" H 8750 13850 50  0001 C CNN
+F 2 "Potentiometer_THT:Potentiometer_Alps_RK09L_Single_Vertical" H 8750 13850 50  0001 C CNN
 F 3 "~" H 8750 13850 50  0001 C CNN
 	1    8750 13850
@@
 F 0 "P_CH2" H 6130 12896 50  0000 R CNN
 F 1 "10k" H 6130 12805 50  0000 R CNN
-F 2 "Potentiometer_THT:Potentiometer_Alps_RK09K_Single_Vertical" H 6200 12850 50  0001 C CNN
+F 2 "Potentiometer_THT:Potentiometer_Alps_RK09L_Single_Vertical" H 6200 12850 50  0001 C CNN
 F 3 "~" H 6200 12850 50  0001 C CNN
 	1    6200 12850
@@
 F 0 "P_CH1" H 4980 12896 50  0000 R CNN
 F 1 "10k" H 4980 12805 50  0000 R CNN
-F 2 "Potentiometer_THT:Potentiometer_Alps_RK09K_Single_Vertical" H 5050 12850 50  0001 C CNN
+F 2 "Potentiometer_THT:Potentiometer_Alps_RK09L_Single_Vertical" H 5050 12850 50  0001 C CNN
 F 3 "~" H 5050 12850 50  0001 C CNN
 	1    5050 12850
@@
 F 0 "P_X1" H 6230 14646 50  0000 R CNN
 F 1 "10k" H 6230 14555 50  0000 R CNN
-F 2 "Potentiometer_THT:Potentiometer_Alps_RK09K_Single_Vertical" H 6300 14600 50  0001 C CNN
+F 2 "Potentiometer_THT:Potentiometer_Alps_RK09L_Single_Vertical" H 6300 14600 50  0001 C CNN
 F 3 "~" H 6300 14600 50  0001 C CNN
 	1    6300 14600
@@
 F 0 "P_CH3" H 7330 12946 50  0000 R CNN
 F 1 "10k" H 7330 12855 50  0000 R CNN
-F 2 "Potentiometer_THT:Potentiometer_Alps_RK09K_Single_Vertical" H 7400 12900 50  0001 C CNN
+F 2 "Potentiometer_THT:Potentiometer_Alps_RK09L_Single_Vertical" H 7400 12900 50  0001 C CNN
 F 3 "~" H 7400 12900 50  0001 C CNN
 	1    7400 12900
@@
 F 0 "P_Y1" H 7430 14646 50  0000 R CNN
 F 1 "10k" H 7430 14555 50  0000 R CNN
-F 2 "Potentiometer_THT:Potentiometer_Alps_RK09K_Single_Vertical" H 7500 14600 50  0001 C CNN
+F 2 "Potentiometer_THT:Potentiometer_Alps_RK09L_Single_Vertical" H 7500 14600 50  0001 C CNN
 F 3 "~" H 7500 14600 50  0001 C CNN
 	1    7500 14600
