File: NanoGris.sch (KiCad schematic (older format))
At the start: 112 parts, among them J10 Conn_01x12, J11 Conn_01x12, J12 Conn_02x05_Odd_Even, J13 Conn_01x10, J14 Conn_01x10, J15 Conn_01x10, J16 Conn_01x03, J7 Conn_01x10, Q1 2N3904, Q2 2N3904, U1 MCP6002_1, U2 MCP6002_1, U3 MCP6002_1, U4 L7805, U5 LM4040LP-5, U6 74HC595, X1 CV_X, Y1 CV_Y

Commit message: Ibom name update
Parts:
- A1: symbol GridsNanoV3-rescue:Arduino_Nano_v2.x-MCU_Module-GridsNanoV2-rescue -> NanoGris-rescue:Arduino_Nano_v2.x-MCU_Module-GridsNanoV2-rescue-GridsNanoV3-rescue
- C1, C10, C12, C16, C2, C3, C4, C5, C6, C7, C8, C9: symbol GridsNanoV3-rescue:C-Device -> NanoGris-rescue:C-Device-GridsNanoV3-rescue
- C11, C13, C14, C15: symbol GridsNanoV3-rescue:CP-Device -> NanoGris-rescue:CP-Device-GridsNanoV3-rescue
- CH1, CH1_AC1, CH1_FILL1, CH2, CH2_AC1, CH2_FILL1, CH3, CH3_AC1, CH3_FILL1, CLK1, CLOCK1, RESET1, RND1, RND2, X1, Y1: symbol GridsNanoV3-rescue:AudioJack2-Connector -> NanoGris-rescue:AudioJack2-Connector-GridsNanoV3-rescue
- D2, D3, D4: symbol GridsNanoV3-rescue:LED-Device -> NanoGris-rescue:LED-Device-GridsNanoV3-rescue
- D5, D6: symbol GridsNanoV3-rescue:D-Device -> NanoGris-rescue:D-Device-GridsNanoV3-rescue
- FID1, FID2: symbol GridsNanoV3-rescue:Fiducial-Mechanical -> NanoGris-rescue:Fiducial-Mechanical-GridsNanoV3-rescue
- H1, H2: symbol GridsNanoV3-rescue:MountingHole-Mechanical -> NanoGris-rescue:MountingHole-Mechanical-GridsNanoV3-rescue
- J10, J11: symbol GridsNanoV3-rescue:Conn_01x12-Connector_Generic -> NanoGris-rescue:Conn_01x12-Connector_Generic-GridsNanoV3-rescue
- J12: symbol GridsNanoV3-rescue:Conn_02x05_Odd_Even-Connector_Generic -> NanoGris-rescue:Conn_02x05_Odd_Even-Connector_Generic-GridsNanoV3-rescue
- J13, J14, J15, J7: symbol GridsNanoV3-rescue:Conn_01x10-Connector_Generic -> NanoGris-rescue:Conn_01x10-Connector_Generic-GridsNanoV3-rescue
- J16: symbol GridsNanoV3-rescue:Conn_01x03-Connector_Generic -> NanoGris-rescue:Conn_01x03-Connector_Generic-GridsNanoV3-rescue
- P_CH1, P_CH2, P_CH3, P_RND1, P_TEMPO1, P_X1, P_Y1: symbol GridsNanoV3-rescue:R_POT-Device -> NanoGris-rescue:R_POT-Device-GridsNanoV3-rescue
- Q1, Q2: symbol GridsNanoV3-rescue:2N3904-Transistor_BJT -> NanoGris-rescue:2N3904-Transistor_BJT-GridsNanoV3-rescue
- R1, R10, R11, R12, R13, R14, R15, R16, R17, R18, R19, R2, R20, R21, R22, R23, R24, R25, R26, R27, R28, R29, R3, R30, R31, R32, R33, R34, R35, R36, R37, R38, R39, R4, R40, R41, R42, R43, R44, R45, R5, R6, R7, R8, R9: symbol GridsNanoV3-rescue:R-Device -> NanoGris-rescue:R-Device-GridsNanoV3-rescue
- RESET2: symbol GridsNanoV3-rescue:SW_Push-Switch -> NanoGris-rescue:SW_Push-Switch-GridsNanoV3-rescue
- U1, U2, U3: symbol GridsNanoV3-rescue:MCP6002-xP-Amplifier_Operational -> NanoGris-rescue:MCP6002-xP-Amplifier_Operational-GridsNanoV3-rescue
- U4: symbol GridsNanoV3-rescue:L7805-Regulator_Linear -> NanoGris-rescue:L7805-Regulator_Linear-GridsNanoV3-rescue
- U5: symbol GridsNanoV3-rescue:LM4040LP-5-Reference_Voltage -> NanoGris-rescue:LM4040LP-5-Reference_Voltage-GridsNanoV3-rescue
- U6: symbol GridsNanoV3-rescue:74HC595-74xx -> NanoGris-rescue:74HC595-74xx-GridsNanoV3-rescue
